File: kicad/sugarboat/sugarboat.kicad_sch (KiCad schematic)
At the start: 45 parts, among them IC1 DW01A, J1 TYPE-C-31-M-12, Q1 FS8205A, Q2 AO3401A, U1 TP4056, U2 MPU-6050, U3 HT7330, U4 E73-2G4M08S1C, U5 SHT30-DIS, Y1 32.768 kHz

Commit message: Renamed KiCad project to sugarboat
Other:
- title: floaty -> sugarboat
Changed lines of the file:
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@@
   (paper "A3")
   (title_block
-    (title "floaty")
+    (title "sugarboat")
     (date "2021-12-29")
     (rev "0.0.1a")
